Commit message: code for new gazebo_harmonic

File: base_robot_description/urdf/arm_gazebo.xacro (robot description, xacro)
@@ -1,27 +1,24 @@
 <?xml version="1.0"?>
 <robot name="my_robot" xmlns:xacro="http://www.ros.org/wiki/xacro">
-    <gazebo reference="arm_base_link">
-        <material>Gazebo/Orange</material>
+    <gazebo>
+        <plugin
+            filename="gz-sim-joint-position-controller-system"
+            name="gz::sim::systems::JointPositionController">
+                <joint_name>arm_base_forearm_joint</joint_name>
+        </plugin>
     </gazebo>
-    <gazebo reference="forearm_link">
-        <material>Gazebo/Yellow</material>
-    </gazebo>
-    <gazebo reference="hand_link">
-        <material>Gazebo/Orange</material>
-    </gazebo>
-    <gazebo>
-         <plugin name="joint_state_publisher_controller"
-            filename="libgazebo_ros_joint_state_publisher.so">
-            <update_rate>10</update_rate>
-            <!-- Name of joints in the model whose states will be published. -->
-            <joint_name>arm_base_forearm_joint</joint_name>
-            <joint_name>forearm_hand_joint</joint_name>
+     <gazebo>
+        <plugin
+            filename="gz-sim-joint-position-controller-system"
+            name="gz::sim::systems::JointPositionController">
+                <joint_name>forearm_hand_joint</joint_name>
         </plugin>
     </gazebo>
     <gazebo>
-        <plugin name="joint_pose_trajectory_controller"
-            filename="libgazebo_ros_joint_pose_trajectory.so">
-            <!-- Update rate in Hz -->
-            <update_rate>2</update_rate>
+        <plugin
+            filename="gz-sim-joint-state-publisher-system"
+            name="gz::sim::systems::JointStatePublisher">
+                <joint_name>arm_base_forearm_joint</joint_name>
+                <joint_name>forearm_hand_joint</joint_name>
         </plugin>
     </gazebo>

File: base_robot_description/urdf/camera_humble.xacro (robot description, xacro)
@@ -30,37 +30,13 @@
     <origin xyz="${(base_length + camera_length) / 2} 0 ${base_height}" rpy="0 0 0"/>
   </joint>
-  <!-- opencv ke liye -->
-  <link name="camera_link_optical"/>
-  <joint name="camera_optical_joint" type="fixed">
-    <parent link="camera_link"/>
-    <child link="camera_link_optical"/>
-    <origin xyz="0 0 0" rpy="${-pi/2} 0 ${-pi/2}"/>
-  </joint>
-  <!-- Gazebo Plugin for Camera -->
-  <gazebo reference ="camera_link">
+  <!-- Gazebo sensor plugin -->
+  <gazebo reference="camera_link">
     <sensor name="camera_sensor" type="camera">
-      <camera>
-        <horizontal_fov>1.0472</horizontal_fov>
-        <image>
-          <width>640</width>
-          <height>480</height>
-          <format>R8G8B8</format>
-        </image>
-        <clip>
-          <near>0.1</near>
-          <far>15.0</far>
-        </clip>
-        <noice>
-          <type>gaussian</type>
-          <mean>0.0</mean>
-          <stddev>0.07</stddev>
-        </noice>
-        <optical_frame_id>camera_link_optical</optical_frame_id>
-        <camera_info_topic>camera/camera_info</camera_info_topic>
-      </camera>
-      <always_on>1</always_on>
-      <update_rate>20.0</update_rate>
+      <pose>0 0 0 0 0 0</pose>
       <visualize>true</visualize>
-      <topic>camera/image_raw</topic>
+      <update_rate>10.0</update_rate>
+      <plugin name="camera_controller" filename="libgazebo_ros_camera.so">
+        <frame_name>camera_link</frame_name>
+      </plugin>
     </sensor>
   </gazebo>
@@ -68,4 +44,2 @@
 <!--
 Gazebo camera and open cv ke liye lec 79 check kar  will be delete after 2025 end-->
-<!--
-opencv ke liye jo frame honi chahiye to y axis se honi chahiye  -->

File: base_robot_description/urdf/mobile_base_gazebo.xacro (robot description, xacro)
@@ -1,38 +1,30 @@
 <?xml version="1.0"?>
-<robot name="my_robot" xmlns:xacro="http://www.ros.org/wiki/xacro">
-    <gazebo reference="base_link">
-        <material>Gazebo/Green</material>
-    </gazebo>
-    <gazebo reference="right_wheel">
-        <material>Gazebo/Grey</material>
-    </gazebo>
-    <gazebo reference="left_wheel">
-        <material>Gazebo/Grey</material>
-    </gazebo>
-    <gazebo reference="caster_wheel">
-        <material>Gazebo/Grey</material>
-        <mu1 value="0.1"/>
-        <mu2 value ="0.1"/>
-    </gazebo>
-    <gazebo>
-         <plugin name="gazebo_ros_diff_drive" filename="libgazebo_ros_diff_drive.so">
-            <!-- Update rate in Hz -->
-            <update_rate>50</update_rate>
-            <!-- wheels -->
-            <left_joint>base_left_wheel_joint</left_joint>
-            <right_joint>base_right_wheel_joint</right_joint>
-            <!-- kinematics -->
-            <wheel_separation>0.45</wheel_separation>
-            <wheel_diameter>0.2</wheel_diameter>
-            <!-- input -->
-            <command_topic>cmd_vel</command_topic>
-            <!-- output -->
-            <publish_odom>true</publish_odom>
-            <publish_odom_tf>true</publish_odom_tf>
-            <publish_wheel_tf>true</publish_wheel_tf>
-            <odometry_topic>odom</odometry_topic>
-            <odometry_frame>odom</odometry_frame>
-            <robot_base_frame>base_footprint</robot_base_frame>
-        </plugin>
-    </gazebo>
+<robot xmlns:xacro="http://www.ros.org/wiki/xacro">
+   <!-- Gazebo friction for a caster wheel (optional) -->
+  <gazebo reference="caster_wheel">
+    <mu1 value="0.1"/>
+    <mu2 value="0.1"/>
+  </gazebo>
+  <!-- DifferentialDrive Plugin -->
+  <gazebo>
+    <plugin
+      filename="gz-sim-diff-drive-system"
+      name="gz::sim::systems::DiffDrive">
+      <left_joint>base_left_wheel_joint</left_joint>
+      <right_joint>base_right_wheel_joint</right_joint>
+      <wheel_separation>0.3</wheel_separation>
+      <wheel_radius>0.05</wheel_radius>
+      <frame_id>odom</frame_id>
+      <child_frame_id>base_footprint</child_frame_id>
+    </plugin>
+  </gazebo>
+  <!-- Joint state publisher -->
+  <gazebo>
+    <plugin
+      filename="gz-sim-joint-state-publisher-system"
+      name="gz::sim::systems::JointStatePublisher">
+      <joint_name>base_left_wheel_joint</joint_name>
+      <joint_name>base_right_wheel_joint</joint_name>
+    </plugin>
+  </gazebo>
 </robot>
